File: 1-5 scale model/Electronics/main-pcb/_autosave-main-pcb.kicad_pcb (KiCad board)
At the start: 2 copper layers, 57 x 73 mm, 21 parts

Commit message: updated it to be better
Routing:
- net Crane_Servo_Yaw: track 0.00 -> 46.8 mm
- net Crane_Servo_Extension: track 0.00 -> 45.5 mm, vias 0 -> 1
- net Crane_Servo_Pitch: track 0.00 -> 42.8 mm
- net L298N_IN1: track 0.00 -> 42.7 mm
- net L298N_IN2: track 0.00 -> 30.4 mm
- net Crane_Limit_Switch: track 0.00 -> 20.9 mm
- net Crane_Servo_Elbow: track 0.00 -> 20.1 mm
Changed lines of the file:
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@@
 	)
 	(segment
-		(start 122 107.5)
-		(end 123.251 106.249)
-		(width 0.2)
-		(layer "F.Cu")
-		(net 6)
-	)
-	(segment
-		(start 123.251 106.249)
-		(end 123.251 95.486892)
+		(start 128 90.737892)
+		(end 128 84)
 		(width 0.2)
 		(layer "F.Cu")
@@
 	)
 	(segment
-		(start 128 90.737892)
-		(end 128 84)
-		(width 0.2)
-		(layer "F.Cu")
-		(net 6)
-	)
-	(segment
-		(start 123.251 95.486892)
+		(start 125 104.5)
+		(end 125 93.737892)
+		(width 0.2)
+		(layer "F.Cu")
+		(net 6)
+	)
+	(segment
+		(start 125 93.737892)
 		(end 128 90.737892)
 		(width 0.2)
@@
 	)
 	(segment
+		(start 122 107.5)
+		(end 125 104.5)
+		(width 0.2)
+		(layer "F.Cu")
+		(net 6)
+	)
+	(segment
+		(start 134 94)
+		(end 134 90.5)
+		(width 0.2)
+		(layer "B.Cu")
+		(net 7)
+	)
+	(segment
+		(start 134 90.5)
+		(end 153 71.5)
+		(width 0.2)
+		(layer "B.Cu")
+		(net 7)
+	)
+	(segment
+		(start 156.5 72.5)
+		(end 153 69)
+		(width 0.2)
+		(layer "B.Cu")
+		(net 8)
+	)
+	(segment
+		(start 134 96.5)
+		(end 141.5 96.5)
+		(width 0.2)
+		(layer "B.Cu")
+		(net 8)
+	)
+	(segment
+		(start 141.5 96.5)
+		(end 156.5 81.5)
+		(width 0.2)
+		(layer "B.Cu")
+		(net 8)
+	)
+	(segment
+		(start 156.5 81.5)
+		(end 156.5 72.5)
+		(width 0.2)
+		(layer "B.Cu")
+		(net 8)
+	)
+	(segment
+		(start 160.5 89)
+		(end 153 81.5)
+		(width 0.2)
+		(layer "F.Cu")
+		(net 9)
+	)
+	(segment
+		(start 169.975 89)
+		(end 160.5 89)
+		(width 0.2)
+		(layer "F.Cu")
+		(net 9)
+	)
+	(segment
+		(start 148 94)
+		(end 149 94)
+		(width 0.2)
+		(layer "F.Cu")
+		(net 10)
+	)
+	(segment
+		(start 138 84)
+		(end 148 94)
+		(width 0.2)
+		(layer "F.Cu")
+		(net 10)
+	)
+	(segment
+		(start 138 81.5)
+		(end 138 84)
+		(width 0.2)
+		(layer "F.Cu")
+		(net 10)
+	)
+	(segment
+		(start 149 94)
+		(end 149.5 93.5)
+		(width 0.2)
+		(layer "F.Cu")
+		(net 10)
+	)
+	(via
+		(at 149.5 93.5)
+		(size 0.6)
+		(drill 0.3)
+		(layers "F.Cu" "B.Cu")
+		(net 10)
+	)
+	(segment
+		(start 169.975 77.5)
+		(end 165.5 77.5)
+		(width 0.2)
+		(layer "B.Cu")
+		(net 10)
+	)
+	(segment
+		(start 165.5 77.5)
+		(end 149.5 93.5)
+		(width 0.2)
+		(layer "B.Cu")
+		(net 10)
+	)
+	(segment
+		(start 163 104)
+		(end 138 79)
+		(width 0.2)
+		(layer "F.Cu")
+		(net 11)
+	)
+	(segment
+		(start 163 105.5)
+		(end 163 104)
+		(width 0.2)
+		(layer "F.Cu")
+		(net 11)
+	)
+	(segment
+		(start 170 112.5)
+		(end 163 105.5)
+		(width 0.2)
+		(layer "F.Cu")
+		(net 11)
+	)
+	(segment
+		(start 139.301 79.301)
+		(end 139.301 77.801)
+		(width 0.2)
+		(layer "F.Cu")
+		(net 12)
+	)
+	(segment
+		(start 169.975 100.5)
+		(end 160.5 100.5)
+		(width 0.2)
+		(layer "F.Cu")
+		(net 12)
+	)
+	(segment
+		(start 160.5 100.5)
+		(end 139.301 79.301)
+		(width 0.2)
+		(layer "F.Cu")
+		(net 12)
+	)
+	(segment
+		(start 139.301 77.801)
+		(end 138 76.5)
+		(width 0.2)
+		(layer "F.Cu")
+		(net 12)
+	)
+	(segment
+		(start 151 89)
+		(end 151 79.5)
+		(width 0.2)
+		(layer "F.Cu")
+		(net 13)
+	)
+	(segment
+		(start 151 79.5)
+		(end 151.5 79)
+		(width 0.2)
+		(layer "F.Cu")
+		(net 13)
+	)
+	(segment
+		(start 157.5 95.5)
+		(end 151 89)
+		(width 0.2)
+		(layer "F.Cu")
+		(net 13)
+	)
+	(segment
+		(start 151.5 79)
+		(end 153 79)
+		(width 0.2)
+		(layer "F.Cu")
+		(net 13)
+	)
+	(segment
