Commit message: balling

File: crew_systems/workspace_analysis/dymaflight/urdf/dymaflight.urdf (robot description, URDF)
Before this commit: robot dymaflight, 8 links, 7 joints
Links:
- added link ee_pos
Joints:
- added joint fixed_j8: type fixed, parent tool_roll, child ee_pos, origin xyz=0 0 0.314325 rpy=0 0 0, axis 0 0 1
